File: BPS-AmperesPCB.kicad_pcb (KiCad board)
At the start: 2 copper layers, 70 x 60 mm, 44 parts, among them J1 Conn_01x04, J2 PeripheralCANConnector, J3 PeripheralCANConnector, U1 PeripheralSOM, U2 INA145UA/2K5, U3 AMC1300BDWV, U4 RO-123.3S_HP

Commit message: edits 1.0 still have to change some stuff Lakshay
Parts:
- moved INP1 1.41 mm to (133.5, 88.6)
- moved OUTN1 1.41 mm to (73.5, 88.6)
- moved GNDPWR1 1.33 mm to (133.6, 39.4)
Routing:
- net GND High: track 0.00 -> 8.66 mm, vias 0 -> 1
- net GND: track 7.82 -> 5.69 mm, vias 0 -> 3
- net /OUTN: track 46.6 -> 47.9 mm, vias 1 -> 2
- net /INP: track 47.1 -> 47.7 mm
Other:
- board text added: "Isolated Power"
- board text added: "Unisolated Power"
- board text removed: "GND GND GND GND GND"
- board text removed: "GND GND GND GND GND GND"
- board text removed: "GND GND GND GND GND GND GND GND GND"
- board text removed: "GND High GND High GND High GND High"
- board text removed: "GND High GND High GND High GND High GND High"
- board text removed: "GND High GND High GND High GND High GND High GND High GND High"
- board text removed: "GNDPWR GNDPWR GNDPWR GNDPWR"
- board text removed: "GNDPWR GNDPWR GNDPWR GNDPWR GNDPWR GNDPWR GNDPWR GNDPWR GNDPWR"

Commit message: gerb'd all over da place
Parts:
- added REF**: Symbol_HighVoltage_Small, UTSVT_Special:Symbol_HighVoltage_Small, F.Cu at (111.0, 90.1)
- moved R9 5.46 mm to (132.0, 55.6), turned to 180 degrees
- moved D1 3.68 mm to (73.3, 60.6)
- moved R5 3.68 mm to (73.3, 63.3)
- moved +3V3H1 2.85 mm to (131.2, 60.4)
- moved +12V1 2.02 mm to (132.2, 47.1)
- moved D4 1.04 mm to (132.0, 53.6)
- moved R2 1.02 mm to (116.2, 55.4)
Routing:
- net GND High: track 8.66 -> 0.00 mm, vias 1 -> 26
- net +3V3 High: track 59.6 -> 52.4 mm
- net Net-(J1-Pin_1): track 20.4 -> 24.8 mm, vias 1 -> 2
- net /OUTN: track 47.9 -> 52.2 mm, vias 2 -> 0
- net +3V3: track 86.5 -> 82.3 mm
- net +12V: track 71.4 -> 69.9 mm, vias 1 -> 2
- net /aOut: track 52.9 -> 51.4 mm
- net /OUTP: track 37.4 -> 38.9 mm
- net GND: track 5.69 -> 4.29 mm, vias 3 -> 31
- net /INN: track 40.0 -> 39.0 mm
- net GNDPWR: vias 0 -> 1
Other:
- board text added: "3v3 High"
- board text added: "Fusebox"
- board text added: "High Voltage Power"
- board text added: "IN"
- board text added: "INN"
- board text added: "INP"
- board text added: "OUT"
- board text added: "OUTN"
- board text added: "OUTP"
- board text added: "aOut (unfiltered)"
- board text removed: "IN N"
- board text removed: "IN P"
- board text removed: "Isolated Power"
- board text removed: "OUT N"
- board text removed: "OUT P"
- board text removed: "SHUNT"
- board text removed: "Unisolated Power"
- board text removed: "VOut"
