File: Peripherals.kicad_sch (KiCad schematic)
At the start: 18 parts, among them J4 SWD, SW1 Reset, U1 STM32L431CBTx, Y1 8M

Commit message: addressed comments
Connections:
- net +3.3V: no longer C12.1, C18.1
- net VDDA: now also C12.1, C18.1
- net I2C1_SCL: no longer names the net of U1.42 (PB6)
- net I2C1_SDA: no longer names the net of U1.43 (PB7)
- net I2C2_PU_En: no longer names the net of U1.29 (PA8)
- net I2C2_SCL: no longer names the net of U1.21 (PB10)
- net I2C2_SDA: no longer names the net of U1.22 (PB11)
- net PA0: no longer names the net of U1.10 (PA0)
- net PA2: no longer names the net of U1.12 (PA2)
- net PB3: no longer names the net of U1.39 (PB3)
- net PB4: no longer names the net of U1.40 (PB4)
- net PB5: no longer names the net of U1.41 (PB5)
- net SPI1_MISO: no longer names the net of U1.16 (PA6)
- net SPI1_MOSI: no longer names the net of U1.17 (PA7)
- net SPI1_NSS: no longer names the net of U1.14 (PA4)
- net SPI1_SCK: no longer names the net of U1.15 (PA5)
- net SPI2_MISO: no longer names the net of U1.27 (PB14)
- net SPI2_MOSI: no longer names the net of U1.28 (PB15)
- net SPI2_NSS: no longer names the net of U1.25 (PB12)
- net SPI2_SCK: no longer names the net of U1.26 (PB13)
- net USART1_RX: no longer names the net of U1.31 (PA10)
- net USART1_TX: no longer names the net of U1.30 (PA9)
Other:
- moved on the sheet: NT1

Commit message: isolated 3v3 done?
Connections:
- net USART1_TX: now reaches U1.30 (PA9)
- net USART1_RX: now reaches U1.31 (PA10)
- no-connect marks 30 -> 28
