File: BPS-AmperesPCB.kicad_sch (KiCad schematic)
At the start: 48 parts, among them IC1 1769205241, IC2 TLV70130DBVR, IC3 1769205241, IC4 TLV70130DBVR, J1 Conn_01x04, J2 PeripheralCANConnector, J3 PeripheralCANConnector, U2 INA145UA/2K5, U3 AMC1300BDWV

Commit message: added 24V buck, bypass caps, more LEDs; started scrutineering circuit and bidirectional current sense
Parts:
- removed +12V1, +3V3, +3V3H1, GND1, GNDH1, GNDPWR1: TestPoint, TestPoint:TestPoint_Keystone_5005-5009_Compact, symbol Connector:TestPoint
- removed C19, C20, C4, C5: 100nF, Capacitor_SMD:C_0805_2012Metric, symbol Device:C
- removed D4: 12V, LED_SMD:LED_0805_2012Metric, symbol Device:LED
- removed D6: 3V3 High, LED_SMD:LED_0805_2012Metric, symbol Device:LED
- removed D7: 3V3, LED_SMD:LED_0805_2012Metric, symbol Device:LED
- removed IC1, IC3: 1769205241, Parts:1769205241, symbol WE_1769205241:1769205241
- removed IC2, IC4: TLV70130DBVR, UTSVT_Power:TLV70130DBVR, symbol utsvt-power:TLV70130DBVR
- removed J2: PeripheralCANConnector, UTSVT_Connectors:Molex_MicroFit3.0_1x4xP3.00mm_PolarizingPeg_Vertical, symbol utsvt-connectors:PeripheralCANConnector
- removed R11, R12, R9: 1.5k, Resistor_SMD:R_0805_2012Metric, symbol Device:R
- added H1, H2: MountingHole, symbol Mechanical:MountingHole
- added IC3: INA241A5IDR, SOIC127P600X175-8N, symbol INA241:INA241A5IDR
- added J1: Discharge V_In, Connector_Molex:Molex_Micro-Fit_3.0_43650-0200_1x02_P3.00mm_Horizontal, symbol Connector_Generic:Conn_01x02
- added J2: Charge V_In, Connector_Molex:Molex_Micro-Fit_3.0_43650-0200_1x02_P3.00mm_Horizontal, symbol Connector_Generic:Conn_01x02
- added J4: PeripheralCAN, UTSVT_Connectors:Molex_Nano-Fit_105309-xx04_1x04_P2.50mm_Vertical, symbol utsvt-connectors:PeripheralCANConnector
- added JP1: Scrutineering, symbol Jumper:Jumper_3_Bridged12
- added R1, R2: ??, Resistor_SMD:R_0805_2012Metric, symbol Device:R
- added TP1: V_In+, TestPoint:TestPoint_Pad_2.0x2.0mm, symbol Connector:TestPoint
- added TP2: V-, TestPoint:TestPoint_Pad_2.0x2.0mm, symbol Connector:TestPoint
- added TP3: V_Out+, TestPoint:TestPoint_Pad_2.0x2.0mm, symbol Connector:TestPoint
- J3: value PeripheralCANConnector -> PeripheralCAN; footprint UTSVT_Connectors:Molex_MicroFit3.0_1x4xP3.00mm_PolarizingPeg_Vertical -> UTSVT_Connectors:Molex_Nano-Fit_105309-xx04_1x04_P2.50mm_Vertical; P/N 436500244 -> 105309-1204
- renumbered C10 to C1, C8 to C3, C7 to C4, C3 to C5, C1 to C6, D2 to D1, D3 to D2, J1 to J5, R8 to R3, R1 to R4, R2 to R5, R3 to R6, R4 to R7, R6 to R8, R7 to R9, U2 to U1, U3 to U2, aOut2 to aOut1
Connections:
- net CAN_HIGH: now also J3.4 (CAN_L), J4.4 (CAN_L); no longer J3.3 (CAN_H)
- net CAN_LOW: now also J3.2 (GND), J4.2 (GND); no longer J3.4 (CAN_L)
- net GNDPWR: now also J3.3 (CAN_H), J4.3 (CAN_H); no longer J3.2 (GNDPWR)
- net +12V renamed +24V
- net +24V: now also J4.1 (24V)
- new net V-: J1.2 (Pin_2), J2.1 (Pin_1), R2.2, TP2.1
- new net V_In+: J1.1 (Pin_1), J2.2 (Pin_2), R1.1, TP1.1
- new net V_Out+: R1.2, R2.1, TP3.1
Other:
- added sheet Power (Power.kicad_sch)
- note added: "- Max current range:"
- note added: "Bidirectional current sense amp"
- note added: "CAN"
- note added: "MCU"
- note added: "Notes"
- note added: "Scrutineering"
- note added: "To-do - pins for status LEDs - verify datasheet values for bypass caps - values for scrutineering + jumper for mode selection - bidirectional current sense - turn into single ended signal before filter"
- note removed: "12V -> 5V DC-DC Converter"
- note removed: "5V -> 3.3V LDO"
- note removed: "Input"
- note removed: "Isolated"
- note removed: "Isolated 3.3 V"
- note removed: "Non-Isolated"
- note removed: "Non-Isolated 3.3 V"
- note removed: "Peripheral Components"
- moved on the sheet: C1, C2, C3, C4, C5, C6, D1, D2, INN1, INP1, J5, OUTN1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
