File: Hardware/USB.kicad_sch (KiCad schematic)
At the start: 0 parts

Commit message: copied USB-C from psom
Parts:
- added C23, C26: 4.7uF, Capacitor_SMD:C_0805_2012Metric_Pad1.18x1.45mm_HandSolder, symbol Device:C
- added C24, C27: 0.1uF, Capacitor_SMD:C_0603_1608Metric_Pad1.08x0.95mm_HandSolder, symbol Device:C
- added C25: 10uF, Capacitor_SMD:C_0805_2012Metric_Pad1.18x1.45mm_HandSolder, symbol Device:C
- added D10: SP0503BAHTG, Package_TO_SOT_SMD:SOT-143, symbol utsvt_ics:SP0503BAH
- added D9: 1N5819HW, Diode_SMD:D_SOD-123, symbol Device:D_Schottky
- added J6: ??, Connector_USB:USB_C_Receptacle_GCT_USB4105-xx-A_16P_TopMnt_Horizontal, symbol Connector:USB_C_Receptacle_USB2.0_16P
- added R15: 1k, Resistor_SMD:R_0603_1608Metric_Pad0.98x0.95mm_HandSolder, symbol Device:R
- added R16: 22k, Resistor_SMD:R_0603_1608Metric_Pad0.98x0.95mm_HandSolder, symbol Device:R
- added R17: 47k, Resistor_SMD:R_0603_1608Metric_Pad0.98x0.95mm_HandSolder, symbol Device:R
- added R18, R19: 5.1k, Resistor_SMD:R_0603_1608Metric_Pad0.98x0.95mm_HandSolder, symbol Device:R
- added U6: CP2102N-A02-GQFN24, UTSVT_ICs:CP2102N-A02-GQFN24, symbol utsvt_ics:CP2102N-Axx-xQFN24
Connections:
- new net +3.3V: C23.1, C24.1, C26.1, C27.1, R15.1, U6.5 (VIO), U6.6 (VDD), U6.7 (VREGIN)
- new net +5V_VBUS: C25.1, D10.4 (K), D9.1 (K), R16.1
- new net CC1: J6.A5 (CC1), R18.1
- new net CC2: J6.B5 (CC2), R19.1
- new net D+: D10.2 (K), J6.A6 (D+), J6.B6 (D+), U6.3 (D+)
- new net D-: D10.3 (K), J6.A7 (D-), J6.B7 (D-), U6.4 (D-)
- new net GND: C23.2, C24.2, C25.2, C26.2, C27.2, D10.1 (A), J6.A1 (GND), J6.A12 (GND), J6.B1 (GND), J6.B12 (GND), J6.S1 (SHIELD), R17.2, R18.2, R19.2, U6.2 (GND), U6.25 (GND)
- new net RST: R15.2, U6.9 (~{RST})
- new net USART1_RX: U6.21 (TXD)
- new net USART1_TX: U6.20 (RXD)
- new net VBUS: R16.2, R17.1, U6.8 (VBUS)
- new net VBUS_IN: D9.2 (A), J6.A4 (VBUS), J6.A9 (VBUS), J6.B4 (VBUS), J6.B9 (VBUS)
- no-connect marks 0 -> 14
Other:
- note added: "CCx Pulldown"
- note added: "Port"
- note added: "TODO: Vertical USB port"
- note added: "UART_TX -> MCU_RX UART_RX <- MCU_TX"
- note added: "USB <-> UART"
- note added: "USB Protection"
- note added: "USB-C"
- note added: "VDD Bypass"
- note added: "VREGIN Bypass"
- note added: "Voltage divider per datasheet pg. 9"
- note added: "shift around for best layout"

Commit message: something changed idk what though
Parts:
- renumbered C23 to C30, C24 to C31, C25 to C32, C26 to C33, C27 to C34, D9 to D11, D10 to D12, J6 to J7, R15 to R20, R16 to R21, R17 to R22, R18 to R23, R19 to R24, U6 to U7
Changed lines of the file:
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@@
 		(dnp no)
 		(fields_autoplaced yes)
-		(property "Reference" "R15"
+		(property "Reference" "R20"
 			(at 137.16 29.2099 0)
 			(effects
@@
 			(project "BPS-AmperesPCB"
 				(path "/a452d214-ea00-440d-a445-5d6103fda43a/c14a2c5c-255b-423f-b086-532f80606e87"
-					(reference "R15")
+					(reference "R20")
 					(unit 1)
 				)
@@
 		(dnp no)
 		(fields_autoplaced yes)
-		(property "Reference" "D9"
+		(property "Reference" "D11"
 			(at 66.3575 27.94 0)
 			(effects
@@
 			(project "BPS-AmperesPCB"
 				(path "/a452d214-ea00-440d-a445-5d6103fda43a/c14a2c5c-255b-423f-b086-532f80606e87"
-					(reference "D9")
+					(reference "D11")
 					(unit 1)
 				)
@@
 		(on_board yes)
 		(dnp no)
-		(property "Reference" "R16"
+		(property "Reference" "R21"
 			(at 125.73 52.578 90)
 			(effects
@@
 			(project "BPS-AmperesPCB"
 				(path "/a452d214-ea00-440d-a445-5d6103fda43a/c14a2c5c-255b-423f-b086-532f80606e87"
-					(reference "R16")
+					(reference "R21")
 					(unit 1)
 				)
@@
 		(on_board yes)
 		(dnp no)
-		(property "Reference" "#PWR061"
+		(property "Reference" "#PWR078"
 			(at 76.2 35.56 0)
 			(effects
@@
 			(project "BPS-AmperesPCB"
 				(path "/a452d214-ea00-440d-a445-5d6103fda43a/c14a2c5c-255b-423f-b086-532f80606e87"
-					(reference "#PWR061")
+					(reference "#PWR078")
 					(unit 1)
 				)
@@
 		(on_board yes)
 		(dnp no)
-		(property "Reference" "#PWR065"
+		(property "Reference" "#PWR082"
 			(at 120.65 52.07 0)
 			(effects
@@
 			(project "BPS-AmperesPCB"
 				(path "/a452d214-ea00-440d-a445-5d6103fda43a/c14a2c5c-255b-423f-b086-532f80606e87"
-					(reference "#PWR065")
+					(reference "#PWR082")
 					(unit 1)
 				)
@@
 		(dnp no)
 		(fields_autoplaced yes)
-		(property "Reference" "R19"
+		(property "Reference" "R24"
 			(at 33.02 104.1399 0)
 			(effects
@@
 			(project "BPS-AmperesPCB"
 				(path "/a452d214-ea00-440d-a445-5d6103fda43a/c14a2c5c-255b-423f-b086-532f80606e87"
-					(reference "R19")
+					(reference "R24")
 					(unit 1)
 				)
@@
 		(dnp no)
 		(fields_autoplaced yes)
-		(property "Reference" "C26"
+		(property "Reference" "C33"
 			(at 101.6 64.7699 0)
 			(effects
@@
 			(project "BPS-AmperesPCB"
 				(path "/a452d214-ea00-440d-a445-5d6103fda43a/c14a2c5c-255b-423f-b086-532f80606e87"
-					(reference "C26")
+					(reference "C33")
 					(unit 1)
 				)
@@
 		(on_board yes)
 		(dnp no)
-		(property "Reference" "#PWR064"
+		(property "Reference" "#PWR081"
 			(at 76.2 53.34 0)
 			(effects
@@
 			(project "BPS-AmperesPCB"
 				(path "/a452d214-ea00-440d-a445-5d6103fda43a/c14a2c5c-255b-423f-b086-532f80606e87"
-					(reference "#PWR064")
+					(reference "#PWR081")
 					(unit 1)
 				)
@@
 		(dnp no)
 		(fields_autoplaced yes)
-		(property "Reference" "D10"
+		(property "Reference" "D12"
 			(at 57.15 104.1399 0)
 			(effects
@@
 			(project "BPS-AmperesPCB"
 				(path "/a452d214-ea00-440d-a445-5d6103fda43a/c14a2c5c-255b-423f-b086-532f80606e87"
-					(reference "D10")
+					(reference "D12")
 					(unit 1)
 				)
@@
 		(on_board yes)
 		(dnp no)
-		(property "Reference" "#PWR070"
+		(property "Reference" "#PWR087"
 			(at 151.13 96.52 0)
 			(effects
@@
 			(project "BPS-AmperesPCB"
 				(path "/a452d214-ea00-440d-a445-5d6103fda43a/c14a2c5c-255b-423f-b086-532f80606e87"
-					(reference "#PWR070")
+					(reference "#PWR087")
 					(unit 1)
 				)
@@
 		(dnp no)
 		(fields_autoplaced yes)
-		(property "Reference" "C24"
+		(property "Reference" "C31"
 			(at 114.3 38.0999 0)
 			(effects
@@
 			(project "BPS-AmperesPCB"
 				(path "/a452d214-ea00-440d-a445-5d6103fda43a/c14a2c5c-255b-423f-b086-532f80606e87"
-					(reference "C24")
+					(reference "C31")
 					(unit 1)
 				)
@@
 		(on_board yes)
 		(dnp no)
-		(property "Reference" "#PWR071"
+		(property "Reference" "#PWR088"
 			(at 53.34 101.6 0)
 			(effects
@@
 			(project "BPS-AmperesPCB"
 				(path "/a452d214-ea00-440d-a445-5d6103fda43a/c14a2c5c-255b-423f-b086-532f80606e87"
-					(reference "#PWR071")
+					(reference "#PWR088")
 					(unit 1)
 				)
@@
 		(dnp no)
 		(fields_autoplaced yes)
-		(property "Reference" "#PWR060"
+		(property "Reference" "#PWR077"
 			(at 153.67 27.94 0)
 			(effects
@@
 			(project "BPS-AmperesPCB"
 				(path "/a452d214-ea00-440d-a445-5d6103fda43a/c14a2c5c-255b-423f-b086-532f80606e87"
-					(reference "#PWR060")
+					(reference "#PWR077")
 					(unit 1)
 				)
@@
 		(dnp no)
 		(fields_autoplaced yes)
-		(property "Reference" "#PWR066"
+		(property "Reference" "#PWR083"
 			(at 97.79 63.5 0)
 			(effects
@@
 			(project "BPS-AmperesPCB"
 				(path "/a452d214-ea00-440d-a445-5d6103fda43a/c14a2c5c-255b-423f-b086-532f80606e87"
-					(reference "#PWR066")
+					(reference "#PWR083")
 					(unit 1)
 				)
@@
 		(dnp no)
 		(fields_autoplaced yes)
-		(property "Reference" "U6"
+		(property "Reference" "U7"
 			(at 153.2733 87.63 0)
 			(effects
@@
 			(project "BPS-AmperesPCB"
 				(path "/a452d214-ea00-440d-a445-5d6103fda43a/c14a2c5c-255b-423f-b086-532f80606e87"
-					(reference "U6")
+					(reference "U7")
 					(unit 1)
 				)
@@
 		(dnp no)
 		(fields_autoplaced yes)
-		(property "Reference" "C25"
+		(property "Reference" "C32"
 			(at 80.01 39.3699 0)
 			(effects
@@
 			(project "BPS-AmperesPCB"
 				(path "/a452d214-ea00-440d-a445-5d6103fda43a/c14a2c5c-255b-423f-b086-532f80606e87"
-					(reference "C25")
+					(reference "C32")
 					(unit 1)
 				)
@@
 		(on_board yes)
 		(dnp no)
-		(property "Reference" "#PWR074"
+		(property "Reference" "#PWR091"
 			(at 50.8 119.38 0)
 			(effects
@@
 			(project "BPS-AmperesPCB"
 				(path "/a452d214-ea00-440d-a445-5d6103fda43a/c14a2c5c-255b-423f-b086-532f80606e87"
-					(reference "#PWR074")
+					(reference "#PWR091")
 					(unit 1)
 				)
@@
 		(dnp no)
 		(fields_autoplaced yes)
-		(property "Reference" "R18"
+		(property "Reference" "R23"
 			(at 22.86 104.1399 0)
 			(effects
@@
 			(project "BPS-AmperesPCB"
 				(path "/a452d214-ea00-440d-a445-5d6103fda43a/c14a2c5c-255b-423f-b086-532f80606e87"
-					(reference "R18")
+					(reference "R23")
 					(unit 1)
 				)
@@
 		(dnp no)
 		(fields_autoplaced yes)
-		(property "Reference" "#PWR062"
+		(property "Reference" "#PWR079"
 			(at 97.79 36.83 0)
 			(effects
@@
 			(project "BPS-AmperesPCB"
 				(path "/a452d214-ea00-440d-a445-5d6103fda43a/c14a2c5c-255b-423f-b086-532f80606e87"
-					(reference "#PWR062")
+					(reference "#PWR079")
 					(unit 1)
 				)
@@
 		(on_board yes)
 		(dnp no)
-		(property "Reference" "#PWR073"
+		(property "Reference" "#PWR090"
 			(at 30.48 118.11 0)
 			(effects
@@
 			(project "BPS-AmperesPCB"
 				(path "/a452d214-ea00-440d-a445-5d6103fda43a/c14a2c5c-255b-423f-b086-532f80606e87"
-					(reference "#PWR073")
+					(reference "#PWR090")
 					(unit 1)
 				)
@@
 		(dnp no)
 		(fields_autoplaced yes)
-		(property "Reference" "C23"
+		(property "Reference" "C30"
 			(at 101.6 38.0999 0)
 			(effects
@@
 			(project "BPS-AmperesPCB"
 				(path "/a452d214-ea00-440d-a445-5d6103fda43a/c14a2c5c-255b-423f-b086-532f80606e87"
-					(reference "C23")
+					(reference "C30")
 					(unit 1)
 				)
@@
 		(on_board yes)
 		(dnp no)
-		(property "Reference" "#PWR063"
+		(property "Reference" "#PWR080"
 			(at 97.79 52.07 0)
 			(effects
@@
 			(project "BPS-AmperesPCB"
 				(path "/a452d214-ea00-440d-a445-5d6103fda43a/c14a2c5c-255b-423f-b086-532f80606e87"
-					(reference "#PWR063")
+					(reference "#PWR080")
 					(unit 1)
 				)
@@
 		(on_board yes)
 		(dnp no)
-		(property "Reference" "#PWR068"
+		(property "Reference" "#PWR085"
 			(at 97.79 78.74 0)
 			(effects
@@
 			(project "BPS-AmperesPCB"
 				(path "/a452d214-ea00-440d-a445-5d6103fda43a/c14a2c5c-255b-423f-b086-532f80606e87"
-					(reference "#PWR068")
+					(reference "#PWR085")
 					(unit 1)
 				)
@@
 		(dnp no)
 		(fields_autoplaced yes)
-		(property "Reference" "J6"
+		(property "Reference" "J7"
 			(at 36.83 26.67 0)
 			(effects
@@
 			(project "BPS-AmperesPCB"
 				(path "/a452d214-ea00-440d-a445-5d6103fda43a/c14a2c5c-255b-423f-b086-532f80606e87"
-					(reference "J6")
+					(reference "J7")
 					(unit 1)
 				)
@@
 		(dnp no)
 		(fields_autoplaced yes)
-		(property "Reference" "C27"
+		(property "Reference" "C34"
 			(at 114.3 64.7699 0)
 			(effects
@@
 			(project "BPS-AmperesPCB"
 				(path "/a452d214-ea00-440d-a445-5d6103fda43a/c14a2c5c-255b-423f-b086-532f80606e87"
-					(reference "C27")
+					(reference "C34")
 					(unit 1)
 				)
@@
 		(on_board yes)
 		(dnp no)
-		(property "Reference" "R17"
+		(property "Reference" "R22"
 			(at 127.635 58.293 0)
 			(effects
@@
 			(project "BPS-AmperesPCB"
 				(path "/a452d214-ea00-440d-a445-5d6103fda43a/c14a2c5c-255b-423f-b086-532f80606e87"
-					(reference "R17")
+					(reference "R22")
 					(unit 1)
 				)
@@
 		(on_board yes)
 		(dnp no)
-		(property "Reference" "#PWR072"
+		(property "Reference" "#PWR089"
 			(at 20.32 118.11 0)
 			(effects
@@
 			(project "BPS-AmperesPCB"
 				(path "/a452d214-ea00-440d-a445-5d6103fda43a/c14a2c5c-255b-423f-b086-532f80606e87"
-					(reference "#PWR072")
+					(reference "#PWR089")
 					(unit 1)
 				)
@@
 		(on_board yes)
 		(dnp no)
-		(property "Reference" "#PWR067"
+		(property "Reference" "#PWR084"
 			(at 132.08 72.39 0)
 			(effects
@@
 			(project "BPS-AmperesPCB"
 				(path "/a452d214-ea00-440d-a445-5d6103fda43a/c14a2c5c-255b-423f-b086-532f80606e87"
-					(reference "#PWR067")
+					(reference "#PWR084")
 					(unit 1)
 				)
@@
 		(on_board yes)
 		(dnp no)
-		(property "Reference" "#PWR069"
+		(property "Reference" "#PWR086"
 			(at 33.02 80.01 0)
 			(effects
@@
 			(project "BPS-AmperesPCB"
 				(path "/a452d214-ea00-440d-a445-5d6103fda43a/c14a2c5c-255b-423f-b086-532f80606e87"
-					(reference "#PWR069")
-					(unit 1)
-				)
+					(reference "#PWR086")
+					(unit 1)
+				)

Commit message: sch almost done
Other:
- note added: "TODO: find vertical port"
- note removed: "TODO: Vertical USB port"
- note removed: "shift around for best layout"
- moved on the sheet: D12, R23, R24
Changed lines of the file:
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@@
 	(paper "A5")
 	(rectangle
-		(start 43.18 86.36)
-		(end 71.12 119.38)
-		(stroke
-			(width 0)
-			(type default)
-		)
-		(fill
-			(type none)
-		)
-	)
-	(rectangle
 		(start 91.44 15.24)
 		(end 193.04 96.52)
@@
 	)
 	(rectangle
-		(start 15.24 86.36)
-		(end 40.64 119.38)
-		(stroke
-			(width 0)
-			(type default)
-		)
-		(fill
-			(type none)
-		)
-	)
-	(rectangle
 		(start 15.24 15.24)
-		(end 86.614 83.82)
+		(end 86.614 121.666)
 		(stroke
 			(width 0)
@@
 		)
 	)
-	(text "shift around for\nbest layout"
-		(exclude_from_sim no)
-		(at 60.706 111.76 0)
-		(effects
-			(font
-				(size 1.27 1.27)
-				(color 255 0 0 1)
-			)
-		)
-	)
 	(text "USB-C"
 		(exclude_from_sim no)
@@
 		)
 	)
-	(text "TODO: Vertical USB port"
+	(text "TODO: find vertical port"
 		(exclude_from_sim no)
 		(at 66.802 71.882 0)
@@
 	(text "CCx Pulldown"
 		(exclude_from_sim no)
-		(at 17.78 88.9 0)
+		(at 20.32 88.9 0)
 		(effects
 			(font
@@
 	(text "USB Protection"
 		(exclude_from_sim no)
-		(at 45.72 88.9 0)
+		(at 48.26 88.9 0)
 		(effects
 			(font
@@
 	(wire
 		(pts
-			(xy 30.48 95.25) (xy 30.48 101.6)
+			(xy 34.29 95.25) (xy 34.29 101.6)
 		)
 		(stroke
@@
 	(wire
 		(pts
-			(xy 50.8 95.25) (xy 50.8 100.33)
+			(xy 57.15 95.25) (xy 57.15 100.33)
 		)
 		(stroke
@@
 	(wire
 		(pts
-			(xy 50.8 110.49) (xy 50.8 113.03)
+			(xy 57.15 110.49) (xy 57.15 113.03)
 		)
 		(stroke
@@
 	(wire
 		(pts
-			(xy 48.26 95.25) (xy 48.26 100.33)
+			(xy 54.61 95.25) (xy 54.61 100.33)
 		)
 		(stroke
@@
 	(wire
 		(pts
-			(xy 20.32 95.25) (xy 20.32 101.6)
+			(xy 24.13 95.25) (xy 24.13 101.6)
 		)
 		(stroke
@@
 	(wire
 		(pts
-			(xy 53.34 97.79) (xy 53.34 100.33)
+			(xy 59.69 97.79) (xy 59.69 100.33)
 		)
 		(stroke
@@
 	(wire
 		(pts
-			(xy 30.48 109.22) (xy 30.48 111.76)
+			(xy 34.29 109.22) (xy 34.29 111.76)
 		)
 		(stroke
@@
 	(wire
 		(pts
-			(xy 20.32 109.22) (xy 20.32 111.76)
+			(xy 24.13 109.22) (xy 24.13 111.76)
 		)
 		(stroke
@@
 	)
 	(label "D+"
-		(at 48.26 95.25 270)
+		(at 54.61 95.25 270)
 		(effects
 			(font
@@
 	)
 	(label "CC1"
-		(at 20.32 95.25 270)
+		(at 24.13 95.25 270)
 		(effects
 			(font
@@
 	)
 	(label "D-"
-		(at 50.8 95.25 270)
+		(at 57.15 95.25 270)
 		(effects
 			(font
@@
 	)
 	(label "CC2"
-		(at 30.48 95.25 270)
+		(at 34.29 95.25 270)
 		(effects
 			(font
@@
 	(symbol
 		(lib_id "Device:R")
-		(at 30.48 105.41 0)
+		(at 34.29 105.41 0)
 		(unit 1)
 		(exclude_from_sim no)
@@
 		(fields_autoplaced yes)
 		(property "Reference" "R24"
-			(at 33.02 104.1399 0)
+			(at 36.83 104.1399 0)
 			(effects
 				(font
@@
 		)
 		(property "Value" "5.1k"
-			(at 33.02 106.6799 0)
+			(at 36.83 106.6799 0)
 			(effects
 				(font
@@
 		)
 		(property "Footprint" "Resistor_SMD:R_0603_1608Metric_Pad0.98x0.95mm_HandSolder"
-			(at 28.702 105.41 90)
+			(at 32.512 105.41 90)
 			(effects
 				(font
@@
 		)
 		(property "Datasheet" "~"
-			(at 30.48 105.41 0)
+			(at 34.29 105.41 0)
 			(effects
 				(font
@@
 		)
 		(property "Description" "Resistor"
-			(at 30.48 105.41 0)
+			(at 34.29 105.41 0)
 			(effects
 				(font
@@
 		)
 		(property "P/N" "CRCW06035K10FKEC "
-			(at 30.48 105.41 0)
+			(at 34.29 105.41 0)
 			(effects
 				(font
@@
 	(symbol
 		(lib_id "utsvt_ics:SP0503BAH")
-		(at 50.8 105.41 0)
+		(at 57.15 105.41 0)
 		(unit 1)
 		(exclude_from_sim no)
@@
 		(fields_autoplaced yes)
 		(property "Reference" "D12"
-			(at 57.15 104.1399 0)
+			(at 63.5 104.1399 0)
 			(effects
 				(font
@@
 		)
 		(property "Value" "SP0503BAHTG"
-			(at 57.15 106.6799 0)
+			(at 63.5 106.6799 0)
 			(effects
 				(font
@@
 		)
 		(property "Footprint" "Package_TO_SOT_SMD:SOT-143"
-			(at 56.515 106.68 0)
+			(at 62.865 106.68 0)
 			(effects
 				(font
@@
 		)
 		(property "Datasheet" "http://www.littelfuse.com/~/media/files/littelfuse/technical%20resources/documents/data%20sheets/sp05xxba.pdf"
-			(at 53.975 102.235 0)
+			(at 60.325 102.235 0)
 			(effects
 				(font
@@
 		)
 		(property "Description" ""
-			(at 50.8 105.41 0)
+			(at 57.15 105.41 0)
 			(effects
 				(font
@@
 		)
 		(property "P/N" "SP0503BAHTG"
-			(at 50.8 105.41 0)
+			(at 57.15 105.41 0)
 			(effects
 				(font
@@
 	(symbol
 		(lib_id "power:+24V")
-		(at 53.34 97.79 0)
+		(at 59.69 97.79 0)
 		(unit 1)
 		(exclude_from_sim no)
@@
 		(dnp no)
 		(property "Reference" "#PWR088"
-			(at 53.34 101.6 0)
+			(at 59.69 101.6 0)
 			(effects
 				(font
@@
 		)
 		(property "Value" "+5V_VBUS"
-			(at 53.086 93.98 0)
+			(at 59.436 93.98 0)
 			(effects
 				(font
@@
 		)
 		(property "Footprint" ""
-			(at 53.34 97.79 0)
+			(at 59.69 97.79 0)
 			(effects
 				(font
@@
 		)
 		(property "Datasheet" ""
-			(at 53.34 97.79 0)
+			(at 59.69 97.79 0)
 			(effects
 				(font
@@
 		)
 		(property "Description" "Power symbol creates a global label with name \"+24V\""
-			(at 53.34 97.79 0)
+			(at 59.69 97.79 0)
 			(effects
 				(font
@@
 	(symbol
 		(lib_id "power:GND")
-		(at 50.8 113.03 0)
+		(at 57.15 113.03 0)
 		(unit 1)
 		(exclude_from_sim no)
@@
 		(dnp no)
 		(property "Reference" "#PWR091"
-			(at 50.8 119.38 0)
+			(at 57.15 119.38 0)
 			(effects
 				(font
@@
 		)
 		(property "Value" "GND"
-			(at 50.8 117.348 0)
+			(at 57.15 117.348 0)
 			(effects
 				(font
@@
 		)
 		(property "Footprint" ""
-			(at 50.8 113.03 0)
+			(at 57.15 113.03 0)
 			(effects
 				(font
@@
 		)
 		(property "Datasheet" ""
-			(at 50.8 113.03 0)
+			(at 57.15 113.03 0)
 			(effects
 				(font
@@
 		)
 		(property "Description" "Power symbol creates a global label with name \"GND\" , ground"
-			(at 50.8 113.03 0)
+			(at 57.15 113.03 0)
 			(effects
 				(font
@@
 	(symbol
 		(lib_id "Device:R")
-		(at 20.32 105.41 0)
+		(at 24.13 105.41 0)
 		(unit 1)
 		(exclude_from_sim no)
@@
 		(fields_autoplaced yes)
 		(property "Reference" "R23"
-			(at 22.86 104.1399 0)
+			(at 26.67 104.1399 0)
 			(effects
 				(font
@@
 		)
 		(property "Value" "5.1k"
-			(at 22.86 106.6799 0)
+			(at 26.67 106.6799 0)
 			(effects
 				(font
@@
 		)
 		(property "Footprint" "Resistor_SMD:R_0603_1608Metric_Pad0.98x0.95mm_HandSolder"
-			(at 18.542 105.41 90)
+			(at 22.352 105.41 90)
 			(effects
 				(font
@@
 		)
 		(property "Datasheet" "~"
-			(at 20.32 105.41 0)
+			(at 24.13 105.41 0)
 			(effects
 				(font
@@
 		)
 		(property "Description" "Resistor"
-			(at 20.32 105.41 0)
+			(at 24.13 105.41 0)
 			(effects
 				(font
@@
 		)
 		(property "P/N" "CRCW06035K10FKEC "
-			(at 20.32 105.41 0)
+			(at 24.13 105.41 0)
 			(effects
 				(font
@@
 	(symbol
 		(lib_id "power:GND")
-		(at 30.48 111.76 0)
+		(at 34.29 111.76 0)
 		(unit 1)
 		(exclude_from_sim no)
@@
 		(dnp no)
 		(property "Reference" "#PWR090"
-			(at 30.48 118.11 0)
+			(at 34.29 118.11 0)
 			(effects
 				(font
@@
 		)
 		(property "Value" "GND"
-			(at 30.48 116.078 0)
+			(at 34.29 116.078 0)
 			(effects
 				(font
@@
 		)
 		(property "Footprint" ""
-			(at 30.48 111.76 0)
+			(at 34.29 111.76 0)
 			(effects
 				(font
@@
 		)
 		(property "Datasheet" ""
-			(at 30.48 111.76 0)
+			(at 34.29 111.76 0)
 			(effects
 				(font
@@
 		)
 		(property "Description" "Power symbol creates a global label with name \"GND\" , ground"
-			(at 30.48 111.76 0)
+			(at 34.29 111.76 0)
 			(effects
 				(font
@@
 	(symbol
 		(lib_id "power:GND")
-		(at 20.32 111.76 0)
+		(at 24.13 111.76 0)
 		(unit 1)
 		(exclude_from_sim no)
@@
 		(dnp no)
 		(property "Reference" "#PWR089"
-			(at 20.32 118.11 0)
+			(at 24.13 118.11 0)
 			(effects
 				(font
@@
 		)
 		(property "Value" "GND"
-			(at 20.32 116.078 0)
+			(at 24.13 116.078 0)
 			(effects
 				(font
@@
 		)
 		(property "Footprint" ""
-			(at 20.32 111.76 0)
+			(at 24.13 111.76 0)
 			(effects
 				(font
@@
 		)
 		(property "Datasheet" ""
-			(at 20.32 111.76 0)
+			(at 24.13 111.76 0)
 			(effects
 				(font
@@
 		)
 		(property "Description" "Power symbol creates a global label with name \"GND\" , ground"
-			(at 20.32 111.76 0)
+			(at 24.13 111.76 0)
 			(effects
 				(font
