File: Hardware/USB.kicad_sch (KiCad schematic)
At the start: 14 parts, among them J5 USB4120-03-C, U9 CP2102N-A02-GQFN24

Commit message: lay out lay out
Parts:
- removed C31: 4.7uF, Capacitor_SMD:C_0603_1608Metric_Pad1.08x0.95mm_HandSolder, symbol Device:C
- removed C33: 10uF, Capacitor_SMD:C_0603_1608Metric_Pad1.08x0.95mm_HandSolder, symbol Device:C
- added C32, C35: 4.7uF, Capacitor_SMD:C_0805_2012Metric_Pad1.18x1.45mm_HandSolder, symbol Device:C
- C34: value 4.7uF -> 10uF; footprint Capacitor_SMD:C_0603_1608Metric_Pad1.08x0.95mm_HandSolder -> Capacitor_SMD:C_0805_2012Metric_Pad1.18x1.45mm_HandSolder; P/N 08055D475KAT4A -> GRM21BR61H106KE43K
- renumbered C32 to C33, C35 to C36, D12 to D13, D13 to D14, U9 to U8
Connections:
- net +3.3V: now also C32.1, C35.1; no longer C34.1
- net +5V_VBUS: now also C34.1
- net GND: now also C32.2, C35.2

Commit message: updated some component part nums
Parts:
- C32, C35: Mfg (none) -> 08055D475KAT4A
- C33, C36: Mfg (none) -> MLASH168SB7104KTNA01
- C34: Mfg (none) -> GRM21BR61H106KE43K
- R19: Mfg (none) -> CRCW06031K00FKEI
- R20: Mfg (none) -> CRCW060322K0FKEAHP; P/N CRCW060322K1FKEBC -> CRCW060322K0FKEAHP
- R21: Mfg (none) -> CRCW060347K0FKECC; P/N CRCW060347K5FKEAHP -> CRCW060347K0FKECC
- R22, R23: Mfg (none) -> CRCW06035K10FKEC
Changed lines of the file:
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@@
+			)
+		)
+		(property "Mfg" "CRCW06031K00FKEI "
+			(at 134.62 30.48 0)
+			(effects
+				(font
+					(size 1.27 1.27)
+				)
+				(hide yes)
 			)
 		)
@@
 			)
 		)
-		(property "P/N" "CRCW060322K1FKEBC "
+		(property "P/N" "CRCW060322K0FKEAHP"
+			(at 125.73 49.53 90)
+			(effects
+				(font
+					(size 1.27 1.27)
+				)
+				(hide yes)
+			)
+		)
+		(property "Mfg" "CRCW060322K0FKEAHP"
 			(at 125.73 49.53 90)
 			(effects
@@
 			)
 		)
+		(property "Mfg" "CRCW06035K10FKEC "
+			(at 34.29 105.41 0)
+			(effects
+				(font
+					(size 1.27 1.27)
+				)
+				(hide yes)
+			)
+		)
 		(pin "1"
 		)
@@
 			)
 		)
+		(property "Mfg" "08055D475KAT4A"
+			(at 97.79 39.37 0)
+			(effects
+				(font
+					(size 1.27 1.27)
+				)
+				(hide yes)
+			)
+		)
 		(pin "1"
 		)
@@
 			)
 		)
+		(property "Mfg" "MLASH168SB7104KTNA01"
+			(at 110.49 39.37 0)
+			(effects
+				(font
+					(size 1.27 1.27)
+				)
+				(hide yes)
+			)
+		)
 		(pin "1"
 		)
@@
 			)
 		)
+		(property "Mfg" "08055D475KAT4A"
+			(at 97.79 66.04 0)
+			(effects
+				(font
+					(size 1.27 1.27)
+				)
+				(hide yes)
+			)
+		)
 		(pin "1"
 		)
@@
 			)
 		)
+		(property "Mfg" "CRCW06035K10FKEC "
+			(at 24.13 105.41 0)
+			(effects
+				(font
+					(size 1.27 1.27)
+				)
+				(hide yes)
+			)
+		)
 		(pin "1"
 		)
@@
 			)
 		)
+		(property "Mfg" "MLASH168SB7104KTNA01"
+			(at 110.49 66.04 0)
+			(effects
+				(font
+					(size 1.27 1.27)
+				)
+				(hide yes)
+			)
+		)
 		(pin "1"
 		)
@@
 			)
 		)
+		(property "Mfg" "GRM21BR61H106KE43K"
+			(at 69.85 44.45 0)
+			(effects
+				(font
+					(size 1.27 1.27)
+				)
+				(hide yes)
+			)
+		)
 		(pin "1"
 		)
@@
 			)
 		)
-		(property "P/N" "CRCW060347K5FKEAHP "
+		(property "P/N" "CRCW060347K0FKECC"
 			(at 132.08 59.69 0)
 			(effects
+				(font
+					(size 1.27 1.27)
+				)
+				(hide yes)
+			)
+		)
+		(property "Mfg" "CRCW060347K0FKECC"
+			(at 132.08 59.69 0)
+			(effects
