File: Hardware/PS-AmperesPCB.kicad_pcb (KiCad board)
At the start: 2 copper layers, 68.9 x 82.5 mm, 158 parts, among them IC1 SN74AHC1G32DBVR, IC2 INA241A4IDR, IC3 AMC1350DWVR, IC4 TLV9002QDRQ1, IC5 LM76202QPWPRQ1, J1 PeripheralCAN, J2 PeripheralCAN, J3 SWD, J4 Conn_01x02_Pin, J5 USB4120-03-C, J6 Scrut Conn, SW1 RST, SW2 BOOT, SW3 Scrutineering, U1 LT1963AEST-3.3#TRPBF, U2 TPS5405DR, U3 TPS2115ADRBR, U4 LT1963AEST-3.3#TRPBF, U5 STM32L431CBTx, U6 TCAN337, U7 CDSOT23-T24CAN, U8 CP2102N-A02-GQFN24, U9 REF35125QDBVR, Y1 8M

Commit message: more routing
Parts:
- SW3: value Scrutineering -> Scrut Select
- moved TP12 7.14 mm to (131.7, 92.3)
- moved D3 6.54 mm to (177.5, 135.3)
- moved D5 6.54 mm to (180.9, 135.3)
- moved R3 6.54 mm to (177.5, 131.6)
- moved R5 6.54 mm to (180.9, 131.6)
- moved D1 6.54 mm to (174.2, 135.3)
- moved R1 6.54 mm to (174.2, 131.6)
- moved D4 6.53 mm to (170.8, 135.3)
- moved R4 6.53 mm to (170.8, 131.6)
- moved TP6 5.59 mm to (164.3, 134.8)
- moved TP7 4.94 mm to (158.5, 134.8)
- moved TP5 4.31 mm to (152.6, 134.8)
- moved TP8 3.70 mm to (146.8, 134.8)
- moved TP3 3.13 mm to (140.9, 134.8)
- moved J4 2.62 mm to (185.1, 104.0), turned to 90 degrees
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Routing:
- net /CAN_LOW: track 2.87 -> 78.7 mm
- net /CAN_HIGH: track 12.7 -> 84.9 mm, vias 0 -> 1
- net +3.3V: track 5.03 -> 58.2 mm, vias 0 -> 23
- net GND: track 0.00 -> 44.6 mm, vias 0 -> 12
- net +5V_VBUS: track 0.00 -> 38.2 mm, vias 0 -> 2
- net /Current Sense/SHUNT-: track 0.00 -> 32.6 mm
- net /Current Sense/SHUNT+: track 0.00 -> 32.2 mm
- net /MCU/Boot_GPIO: track 0.00 -> 27.0 mm, vias 0 -> 2
- net /CAN/CAN1_TX: track 0.00 -> 24.2 mm, vias 0 -> 1
- net /CAN/CAN1_RX: track 0.00 -> 20.7 mm, vias 0 -> 1
- net +5V_BUCK: track 0.00 -> 20.4 mm, vias 0 -> 5
- net +3.3V HV: track 2.61 -> 22.9 mm, vias 0 -> 9
- net /MCU/SWCLK: track 0.00 -> 20.0 mm
- net +24V: track 0.00 -> 18.4 mm, vias 0 -> 2
- net /MCU/USART1_RX: track 0.00 -> 17.1 mm, vias 0 -> 2
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- added copper zone on B.Cu, net +3.3V
- added copper zone on B.Cu, net +3.3V HV
- added copper zone on B.Cu, net /Power/PowerProtection/RTN
Other:
- board size 68.9 x 82.5 mm -> 81.4 x 95.6 mm

Commit message: more routing
Parts:
- added TP15: GND, TestPoint:TestPoint_Pad_1.0x1.0mm, F.Cu at (180.8, 135.1)
- moved D4 27.0 mm to (152.0, 115.9), turned to 0 degrees
- moved R4 25.8 mm to (152.0, 114.0), turned to 0 degrees
- moved R1 22.9 mm to (151.4, 133.4), turned to 0 degrees
- moved D1 22.8 mm to (151.4, 135.3), turned to 0 degrees
- moved R3 16.4 mm to (161.2, 133.3), turned to 0 degrees
- moved D3 16.2 mm to (161.3, 135.3), turned to 0 degrees
- moved TP7 8.83 mm to (167.3, 135.1)
- moved TP6 7.98 mm to (172.3, 135.1)
- moved TP3 6.55 mm to (147.4, 135.1)
- moved R5 5.22 mm to (176.0, 133.3), turned to 0 degrees
- moved TP5 4.98 mm to (157.6, 135.1)
- moved D5 4.88 mm to (176.0, 135.3), turned to 0 degrees
- moved TP8 4.55 mm to (142.2, 135.1)
- moved D2 3.28 mm to (149.2, 80.4), turned to 0 degrees
- moved R2 1.49 mm to (149.2, 82.1), turned to 0 degrees
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Routing:
- net /MCU/ADC1_IN16: track 2.60 -> 111.6 mm, vias 0 -> 2
- net GND: track 44.6 -> 86.0 mm, vias 12 -> 18
- net /Current Sense/Scrut-: track 10.7 -> 46.0 mm, vias 0 -> 2
- net /Current Sense/Scrut_Out: track 5.62 -> 36.8 mm, vias 0 -> 2
- net /Current Sense/Scrut+: track 6.40 -> 34.4 mm, vias 0 -> 2
- net /Current Sense/SHUNT+: track 32.2 -> 54.2 mm, vias 0 -> 2
- net /Current Sense/SHUNT-: track 32.6 -> 49.1 mm, vias 0 -> 2
- net /CAN_LOW: track 78.7 -> 88.2 mm, vias 0 -> 1
- net +5V: track 5.39 -> 13.8 mm
- net +5V_VBUS: track 38.2 -> 45.4 mm, vias 2 -> 7
- net /USB/D-: track 8.97 -> 13.4 mm, vias 0 -> 2
- net GNDA: track 4.88 -> 8.36 mm, vias 0 -> 1
- net VDDA: track 5.44 -> 8.29 mm, vias 0 -> 1
- net /Power/PWR_Fault: track 4.71 -> 7.57 mm, vias 0 -> 2
- net /Power/STAT: track 0.00 -> 2.67 mm
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- added copper zone on F.Cu, net +3.3V
- added copper zone on B.Cu, net +5V_VBUS
- added copper zone on B.Cu, net /USB/VBUS_IN
- removed copper zone on F.Cu, net +5V
Other:
- board size 81.4 x 95.6 mm -> 81.8 x 95.6 mm

Commit message: review council
Parts:
- C6: moved to B.Cu
- moved C6 31.3 mm to (195.8, 117.4), turned to 180 degrees
- moved R7 3.25 mm to (157.0, 123.7), turned to -90 degrees
- moved C8 1.64 mm to (159.3, 117.5), turned to 90 degrees
- moved C7 1.63 mm to (157.1, 117.3), turned to 90 degrees
- moved C12 1.48 mm to (159.2, 123.7), turned to -90 degrees
Routing:
- net GND: track 86.0 -> 72.1 mm, vias 18 -> 19
- net +5V_VBUS: track 45.4 -> 38.3 mm
- net Net-(U2-BOOT): track 3.04 -> 0.00 mm
- net Net-(D6-K): track 3.00 -> 0.00 mm
- net /Power/ROSC: track 3.04 -> 5.49 mm
- net /Power/ILIM: track 2.45 -> 0.03 mm, vias 2 -> 0
- net +1V25: vias 0 -> 2
- added copper zone on B.Cu, net GND

Commit message: silkscreen work
Parts:
- C6: moved to F.Cu
- R31: value 24m -> 19K
- SW3: value Scrut Select -> Scrutineering
- TP1: value TP_Current -> I_Out
- TP6: value 5V_BK -> 5V_Buck
- moved LOGO1 97.7 mm to (184.3, 129.6)
- moved C6 27.6 mm to (168.2, 116.4), turned to 0 degrees
- moved D6 6.72 mm to (175.3, 114.7), turned to 90 degrees
- moved R36 4.31 mm to (135.4, 121.6), turned to -90 degrees
- moved D4 2.15 mm to (154.1, 115.6)
- moved R4 2.15 mm to (154.1, 113.7)
- moved C13 1.81 mm to (171.6, 122.4)
- moved R6 1.75 mm to (171.6, 120.7)
- moved R37 1.69 mm to (137.5, 122.3), turned to -90 degrees
- moved R38 1.25 mm to (139.5, 122.3), turned to -90 degrees
- moved D16 1.24 mm to (188.1, 66.8)
- moved D15 1.24 mm to (188.0, 69.4)
- moved D10 0.88 mm to (171.7, 70.8)
- moved R14 0.88 mm to (171.7, 74.9)
- moved D9 0.59 mm to (175.0, 70.8)
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- renumbered R39 to SHUNT
Routing:
- net +3.3V: track 60.1 -> 114.4 mm
- net GND: track 72.1 -> 62.1 mm, vias 19 -> 23
- net Net-(U2-BOOT): track 0.00 -> 6.52 mm
- net /MCU/Boot_GPIO: track 27.7 -> 22.2 mm, vias 2 -> 4
- net +5V HV: track 0.00 -> 4.70 mm, vias 0 -> 4
- net /Power/ILIM: track 0.03 -> 2.45 mm
- net /Power/PowerProtection/UVLO: track 6.15 -> 8.06 mm
- net /Current Sense/I_OUT: track 29.9 -> 31.8 mm
- net +5V_BUCK: track 21.8 -> 23.5 mm
- net +24V: track 20.3 -> 18.6 mm
- net /MCU/ADC1_IN16: track 111.6 -> 113.1 mm
- net /Power/PWR_Fault: track 7.57 -> 8.81 mm
- net Net-(IC1-A): track 5.09 -> 6.25 mm, vias 0 -> 2
- net /CAN/Fault: track 7.62 -> 8.78 mm
- net /Current Sense/Scrut-: track 46.0 -> 47.1 mm
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- added copper zone on B.Cu, net +5V HV
- removed copper zone on F.Cu, net +5V HV
Other:
- board text added: "100uH"
- board text added: "BOOT"
- board text added: "CAN"
- board text added: "Current Signal"
- board text added: "High Voltage"
- board text added: "LM7620"
- board text added: "LT1963AEST"
- board text added: "Low Voltage"
- board text added: "Peripheral CAN"
- board text added: "Reset"
- board text added: "Shunt -- Scrut"
- board text added: "TPS405DR"
- board text added: "TVS"
- board text added: "Term"
- board text added: "USB"
- board text removed: "AAHAHAH"

Commit message: added models
Parts:
- removed SHUNT: WSBS8518L2500JTP3, Parts:WSBS8518L2500JKM4
- added R39: WSBS8518L2500JTP3, Parts:WSBS8518L2500JKM4, F.Cu at (115.7, 70.1)
- added TP16: 1V25, TestPoint:TestPoint_Pad_1.0x1.0mm, F.Cu at (131.7, 96.2)
- SW3: value Scrutineering -> Scrut Select
- TP3: value 24V -> - 24V -
- TP5: value 3V3 -> - 3V3 -
- TP6: value 5V_Buck -> 5V_BK
- moved R4 6.75 mm to (152.7, 120.3), turned to -90 degrees
- moved D4 6.59 mm to (154.5, 122.1), turned to 90 degrees
- moved C33 3.11 mm to (164.7, 87.5), turned to -90 degrees
- moved C36 2.96 mm to (164.7, 84.0), turned to 90 degrees
- moved C54 2.16 mm to (151.7, 122.9)
- moved R32 1.87 mm to (151.7, 124.7)
- moved R33 1.85 mm to (150.8, 120.3), turned to -90 degrees
- moved R31 1.59 mm to (151.7, 126.5)
- moved H1 1.19 mm to (189.2, 61.0)
- moved R30 1.17 mm to (151.7, 128.2)
- moved R19 1.12 mm to (165.7, 84.9)
- moved R20 1.12 mm to (165.7, 88.7)
- moved R21 1.12 mm to (165.7, 86.8)
- moved R22 1.12 mm to (161.0, 99.2)
- moved U8 1.12 mm to (161.0, 84.9)
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Routing:
- net +1V25: track 15.1 -> 28.2 mm, vias 2 -> 4
- net GND: track 62.1 -> 56.5 mm, vias 23 -> 22
- net /USB/VBUS_IN: track 9.78 -> 5.05 mm
- net +3.3V: track 114.4 -> 110.3 mm
- net /MCU/USART1_RX: track 17.7 -> 20.3 mm
- net /MCU/USART1_TX: track 17.2 -> 19.7 mm
- net +5V_VBUS: track 38.7 -> 40.2 mm, vias 6 -> 8
- net /Power/PWR_Fault: track 8.81 -> 7.42 mm, vias 2 -> 0
- net Net-(IC5-DVDT): track 3.93 -> 2.85 mm
- net /MCU/ADC1_IN16: track 113.1 -> 113.8 mm
- net /Power/PowerProtection/IMON: track 5.94 -> 6.53 mm
- net /Power/PowerProtection/RTN: track 11.1 -> 10.5 mm
Other:
- board size 81.8 x 95.6 mm -> 81.4 x 95.2 mm
- board text added: "1V25"
- board text added: "3.3V"
- board text added: "AMC1350"
- board text added: "Clk"
- board text added: "GND"
- board text added: "IO"
- board text added: "PWR Fault"
- board text added: "TLV9002"

Commit message: i don't know what I changed
Other:
- board size 81.4 x 95.2 mm -> 81.8 x 95.6 mm
