File: Hardware/CAN.kicad_sch (KiCad schematic)
At the start: 10 parts, among them J4 Conn_01x02_Pin, U6 TCAN337, U7 CDSOT23-T24CAN

Commit message: docs, bom pushed
Parts:
- J4: P/N 1053091202 -> (none)
Changed lines of the file:
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@@
-			)
-		)
-		(property "P/N" "1053091202"
-			(at 107.95 77.47 0)
-			(effects
-				(font
-					(size 1.27 1.27)
-				)
-				(hide yes)
 			)
 		)
